Commit message: Add project5 files

File: my_robot/urdf/my_robot.xacro (robot description, xacro)
@@ -159,4 +159,11 @@
     <material>Gazebo/SkyBlue</material>
   </gazebo>
+  <joint name="camera_optical_joint" type="fixed">
+    <origin xyz="0 0 0" rpy="-1.5707 0 -1.5707"/>
+    <parent link="camera"/>
+    <child link="camera_link_optical"/>
+  </joint>
+  <link name="camera_link_optical">
+  </link>
   <joint type="fixed" name="hokuyo_joint">
     <origin xyz="0.12 0 0.08" rpy="0 0 0"/>
